File: hm2.kicad_sch (KiCad schematic)
At the start: 0 parts

Commit message: schematics: Placing symbols
Parts:
- added C?: 1nF, symbol Device:C
- added C? (x5): 47nF, symbol Device:C
- added C? (x3): 47uF, symbol Device:C_Polarized
- added C?: 10uF, symbol Device:C_Polarized
- added C? (x2): 10pF, symbol Device:C
- added C? (x2): 1uF, symbol Device:C_Polarized
- added D? (x5): 1N4148, Diode_THT:D_DO-35_SOD27_P7.62mm_Horizontal, symbol Diode:1N4148
- added D? (x2): Ge. Diode, symbol Device:D
- added H? (x4): MountingHole_Pad, symbol Mechanical:MountingHole_Pad
- added J? (x2): Conn_01x01, symbol Connector_Generic:Conn_01x01
- added Q?: 2SC2240, Package_TO_SOT_THT:TO-92_Inline, symbol Transistor_BJT:2SC1815
- added Q?: BF245A, Package_TO_SOT_THT:TO-92_Inline, symbol Transistor_FET:BF245A
- added Q?: Q_PNP_BCE, symbol Device:Q_PNP_BCE
- added R?: 22, symbol Device:R
- added R? (x10): 10k, symbol Device:R
- added R?: 1M, symbol Device:R
- added R?: 22k, symbol Device:R
- added R? (x3): 100k, symbol Device:R
- added R?: 1k, symbol Device:R
- added R?: 68k, symbol Device:R
- added R?: 150, symbol Device:R
- added R?: 220k, symbol Device:R
- added R?: 120, symbol Device:R
- added R?: 470k, symbol Device:R
- added R?: 47k, symbol Device:R
- added RV? (x2): 250k log, symbol Device:R_Potentiometer
Connections:
- new net: Q?.1 (E), R?.2
- new net: J?.1 (Pin_1), R?.1
- new net: C?.1, R?.2 (x2)
- new net: D?.1 (K), D?.2 (A)
- new net: C?.2, D?.1 (K), D?.2 (A), R?.2
- new net: R?.2, RV?.1
- new net: J?.1 (Pin_1), RV?.2
- new net: C?.1, C?.2, C?.2, Q?.2 (C), R?.1, R?.2
- new net: C?.1, Q?.3 (B), R?.1, R?.2, R?.2
- new net: C?.1, R?.2, R?.2, R?.2, R?.2 (x2)
- new net: C?.2, Q?.1 (G), R?.1
- new net: C?.2, C?.2, D?.1 (K), D?.2 (A), R?.2
- new net: C?.2, R?.1 (x3)
- new net: R?.1, RV?.1
- new net: R?.2, RV?.3
- new net: C?.1, Q?.1 (B), R?.1, R?.1, R?.2
- new net: C?.1, Q?.2 (S), R?.2
- new net: C?.1, C?.2, D?.1 (K), D?.2 (A), R?.1
- new net: C?.2, Q?.2 (C), R?.1, R?.2, R?.2
- new net: D?.1 (K), D?.2 (A), R?.2
- new net: D?.1 (K), D?.2 (A), R?.1
- new net: C?.1, R?.1 (x2)
- new net: Q?.3 (E), R?.1
- new net +9V: Q?.3 (D), R?.1, R?.1
- new net GND: C?.1, C?.2, C?.2, D?.1 (K), D?.2 (A), H?.1, H?.1, H?.1, H?.1, R?.1, R?.1, R?.1, R?.1, R?.1, RV?.2, RV?.3
